Commit message: visualize the case of grasping small poll

File: robots/hydrus/urdf/common.xacro (robot description, xacro)
@@ -7,5 +7,5 @@
   <!-- kinematics [m] -->
   <xacro:property name="link_length" value=".6" />
-  <xacro:property name="protector_radius" value=".1925" />
+  <xacro:property name="protector_radius" value=".1025" />
   <xacro:property name="head_leg_offset" value="${0.3 - 0.25884}" />
   <xacro:property name="end_leg_offset" value="${0.3 + 0.25884}" />
