Commit message: circle shaped dragon's urdf

File: robots/dragon/robots/octa/euclid_201709.urdf.xacro (robot description, xacro)
@@ -8,4 +8,8 @@
   <xacro:dragon_one_rotor_module self="2" child="3" baselink="true" />
   <xacro:dragon_one_rotor_module self="3" child="4" baselink="false" />
-  <xacro:dragon_one_rotor_module self="4" child="4" baselink="false" />
+  <xacro:dragon_one_rotor_module self="4" child="5" baselink="false" />
+  <xacro:dragon_one_rotor_module self="5" child="6" baselink="false" />
+  <xacro:dragon_one_rotor_module self="6" child="7" baselink="false" />
+  <xacro:dragon_one_rotor_module self="7" child="8" baselink="false" />
+  <xacro:dragon_one_rotor_module self="8" child="8" baselink="false" />
 </robot>

File: robots/dragon/urdf/dragon_common.xacro (robot description, xacro)
@@ -36,7 +36,7 @@
     -->
     <visual>
-      <origin rpy="0 0 0" xyz="${link_length* 0.5} 0 0"/>
+      <origin rpy="0 0 0" xyz="0 -0.2 -0.05"/>
       <geometry>
-        <mesh filename="package://dragon/urdf/mesh/ducted_fan_${type}.dae"/>
+        <mesh filename="package://dragon/urdf/mesh/ducted_fan_${type}_spine_shaped.dae"/>
       </geometry>
     </visual>
