Commit message: [DRAGON] [gakushin_fig] show spine in link (not change the original spine) and write test urdf code

File: robots/dragon/urdf/dragon_spine_based_link.urdf.xacro (robot description, xacro)
@@ -1,7 +1,9 @@
 <?xml version="1.0"?>
 <robot
-    xmlns:xacro="http://www.ros.org/wiki/xacro" name="dragon_one_rotor_link" >
+    xmlns:xacro="http://www.ros.org/wiki/xacro" name="dragon_spine_based_link" >
   <!-- D-H kai description(different from prof.nakamura) -->
-  <xacro:macro name="dragon_one_rotor_module" params="self child baselink">
+  <xacro:include filename="$(find dragon)/urdf/dragon_common.xacro" />
+  <xacro:include filename="$(find dragon)/urdf/dragon_spine_assy.urdf.xacro" />
+  <xacro:macro name="dragon_one_rotor_module" params="self child baselink pitch yaw">
     <!-- link -->
     <link name="link${self}">
@@ -84,4 +86,7 @@
     </link>
     <xacro:damping_factor link ="link${self}"/>
+    <!-- spine link -->
+    <!-- connected to next child link -->
+    <xacro:dragon_spine_assy whole="${self}" whole_child="${child}" pitch="${pitch}" yaw="${yaw}"/>
     <!-- gimbal roll -->
     <joint name="gimbal${self}_roll" type="revolute">
@@ -199,44 +204,4 @@
     </link>
     <xacro:damping_factor link ="thrust${self}"/>
-    <!-- joint -->
-    <xacro:unless value="${self == child}">
-      <joint name="joint${self}_pitch" type="revolute">
-        <limit effort="10.0" lower="${-pi/2}" upper="${pi/2}" velocity="0.1"/>
-        <parent link="link${self}"/>
-        <child link="inter_joint${self}"/>
-        <origin rpy="0 0 0" xyz="${link_length} 0 0"/>
-        <axis xyz="0 1 0"/>
-        <dynamics damping="0.9" friction="0.05"/>
-      </joint>
-      <!-- inter joint -->
-      <link name="inter_joint${self}">
-        <!-- common inertial -->
-        <inertial>
-          <origin xyz="${inter_joint_x_offset + 3.43 * 0.001} ${-4.27 * 0.001} ${-1.55 * 0.001}" rpy="0 0 0"/>
-          <mass value="0.1329" />
-          <inertia
-              ixx="0.0001" iyy="0.0001" izz="0.0001"
-              ixy="0" ixz="0.0" iyz="0.0"/>
-        </inertial>
-        <visual>
-          <origin rpy="0 0 0" xyz="${inter_joint_x_offset} 0 0"/>
-          <geometry>
-            <mesh filename="package://dragon/urdf/mesh/inter_joint_junction.dae"/>
-          </geometry>
-        </visual>
-      </link>
-      <joint name="joint${self}_yaw" type="revolute">
-        <limit effort="10.0" lower="${-pi}" upper="${pi}" velocity="0.1"/>
-        <parent link="inter_joint${self}"/>
-        <child link="link${child}"/>
-        <origin rpy="0 0 0" xyz="${2 * inter_joint_x_offset} 0 0"/>
-        <axis xyz="0 0 1"/>
-        <dynamics damping="0.9" friction="0.05"/>
-      </joint>
-      <gazebo reference="inter_joint${self}">
-        <mu1>0.2</mu1>
-        <mu2>0.2</mu2>
-      </gazebo>
-    </xacro:unless>
     <xacro:if value="${self == 1}">
       <!-- dummy root link for KDL -->
