Commit message: [REFACTORING] change indentation of dragon_common.xacro to show them clearly

File: robots/dragon/urdf/dragon_common.xacro (robot description, xacro)
@@ -22,8 +22,8 @@
     <!-- box collision geometry does not work well for FCL -->
     <collision>
-    <origin rpy="0 0 0" xyz="${link_length* 0.5} 0 0"/>
-    <geometry>
-    <box size="${link_length} 0.15 0.1686"/>
-    </geometry>
+      <origin rpy="0 0 0" xyz="${link_length* 0.5} 0 0"/>
+      <geometry>
+        <box size="${link_length} 0.15 0.1686"/>
+      </geometry>
     </collision>
     <!-- cylinder collision geometry works well for FCL

Commit message: [DRAGON][gakushin_fig] show spine link with outside of rotor

File: robots/dragon/urdf/dragon_common.xacro (robot description, xacro)
@@ -14,5 +14,5 @@
   <xacro:property name="inter_joint_x_offset" value=".02575" />
   <xacro:property name="gimbal_roll_x_offset" value="-0.01" />
-  <xacro:property name="gimbal_pitch_z_offset" value="0.037" />
+  <xacro:property name="gimbal_pitch_z_offset" value="0.033" />
   <!-- dynamics -->
   <m_f_rate value="0" /> <!-- drug torque rate -->
@@ -35,10 +35,4 @@
     </collision>
     -->
-    <visual>
-      <origin rpy="0 0 0" xyz="0 -0.2 -0.05"/>
-      <geometry>
-        <mesh filename="package://dragon/urdf/mesh/ducted_fan_${type}_spine_shaped.dae"/>
-      </geometry>
-    </visual>
   </xacro:macro>
   <!-- friction -->

File: robots/dragon/urdf/dragon_spine_based_link.urdf.xacro (robot description, xacro)
@@ -94,5 +94,5 @@
       <parent link="link${self}"/>
       <child link="gimbal${self}_roll_module"/>
-      <origin rpy="0 0 0" xyz="${link_length/2} -0.22 0"/>
+      <origin rpy="0 0 ${pi/2}" xyz="0.02 -0.02 0"/>
       <axis xyz="1 0 0"/>
       <dynamics damping="0.1" friction="0.0"/>
@@ -107,7 +107,7 @@
       </inertial>
       <visual>
-        <origin xyz="${gimbal_roll_x_offset} 0.1 0" rpy="0 0 0"/>
+        <origin xyz="${gimbal_roll_x_offset} 0 0" rpy="0 0 0"/>
         <geometry>
-          <mesh filename="package://dragon/urdf/mesh/ducted_fan_gimbal_roll.dae"/>
+          <mesh filename="package://dragon/urdf/mesh/ducted_fan_gimbal_roll_spine.dae"/>
         </geometry>
       </visual>
@@ -133,5 +133,5 @@
       <parent link="gimbal${self}_roll_module"/>
       <child link="gimbal${self}_pitch_module"/>
-      <origin rpy="0 0 0" xyz="0 0 ${gimbal_pitch_z_offset}"/>
+      <origin rpy="0 0 0" xyz="-0.07 0 ${gimbal_pitch_z_offset}"/>
       <axis xyz="0 1 0"/>
       <dynamics damping="0.1" friction="0.0"/>
@@ -146,7 +146,7 @@
       </inertial>
       <visual>
-        <origin xyz="0.05 0.1 -0.05" rpy="0 0 3.14"/>
+        <origin xyz="0 0 0" rpy="0 0 0"/>
         <geometry>
-          <mesh filename="package://dragon/urdf/mesh/ducted_fan_single_rotor.dae" scale="0.001 0.001 0.001"/>
+          <mesh filename="package://dragon/urdf/mesh/ducted_fan_gimbal_pitch.dae"/>
         </geometry>
       </visual>

Commit message: [DRAGON][gakushin_fig][debug] delete link_model's collision check

File: robots/dragon/urdf/dragon_common.xacro (robot description, xacro)
@@ -20,19 +20,4 @@
   <xacro:property name="min_force" value="2" /> <!-- [N] -->
   <xacro:macro name="link_model" params="type">
-    <!-- box collision geometry does not work well for FCL -->
-    <collision>
-      <origin rpy="0 0 0" xyz="${link_length* 0.5} 0 0"/>
-      <geometry>
-        <box size="${link_length} 0.15 0.1686"/>
-      </geometry>
-    </collision>
-    <!-- cylinder collision geometry works well for FCL
-    <collision>
-      <origin rpy="0 ${pi/2} 0" xyz="${link_length* 0.5} 0 0"/>
-      <geometry>
-        <cylinder length="${link_length}" radius="0.06" />
-      </geometry>
-    </collision>
-    -->
   </xacro:macro>
   <!-- friction -->
