Commit message: [DRAGON][gakushin_fig][debug] change the end joint of the link to fig the link

File: robots/dragon/urdf/dragon_spine_assy.urdf.xacro (robot description, xacro)
@@ -60,5 +60,5 @@
         <parent link="spinelink${whole_link}_${self}"/>
         <child link="link${whole_link_child}"/>
-        <origin xyz="${spine_length} 0 0" rpy="0 0 0" />
+        <origin xyz="${spine_length+.01} 0 0" rpy="0 0 0" />
       </joint>
     </xacro:if>

Commit message: [DRAGON][gakushin_fig][debug] can rotate roll direction of spine

File: robots/dragon/urdf/dragon_spine_assy.urdf.xacro (robot description, xacro)
@@ -57,8 +57,11 @@
     </xacro:unless>
     <xacro:if value="${self == child and whole_link!=whole_link_child}">
-      <joint name="spine_${whole_link}_end_joint" type="fixed" >
+      <joint name="spine_${whole_link}_end_joint" type="revolute" >
+        <limit effort="3" lower="-3.14" upper="3.14" velocity="12.5"/>
         <parent link="spinelink${whole_link}_${self}"/>
         <child link="link${whole_link_child}"/>
         <origin xyz="${spine_length+.01} 0 0" rpy="0 0 0" />
+        <axis xyz="1 0 0"/>
+        <dynamics damping="0.1" friction="0.0"/>
       </joint>
     </xacro:if>
