Commit message: [agile_multirotor] urdf model for tello flight

File: robots/mini_quadrotor/urdf/robot.urdf.xacro (robot description, xacro)
@@ -6,7 +6,7 @@
   <thrust_link name="thrust" />
   <!-- kinematics [m] -->
-  <xacro:property name="rotor_x" value="0.085" />
-  <xacro:property name="rotor_y" value="0.085" />
-  <xacro:property name="rotor_z" value="0.026" />
+  <xacro:property name="rotor_x" value="0.035" />
+  <xacro:property name="rotor_y" value="0.035" />
+  <xacro:property name="rotor_z" value="0.010" />
   <!-- dynamics -->
   <m_f_rate value="-0.011" /> <!-- drag torque rate -->
@@ -49,9 +49,9 @@
       <inertial>
         <origin xyz="0 0 0" rpy="0 0 0"/>
-        <mass value="0.0091"/>
+        <mass value="0.00091"/>
         <inertia
-            ixx="0.00000807" ixy="0.0" ixz="0.0"
-            iyy="0.00000807" iyz="0.0"
-            izz="0.00001612"/>
+            ixx="0.0000000807" ixy="0.0" ixz="0.0"
+            iyy="0.0000000807" iyz="0.0"
+            izz="0.0000001612"/>
       </inertial>
       <visual>
@@ -80,9 +80,9 @@
     <inertial>
       <origin xyz="0 0 0" rpy="0 0 0"/>
-      <mass value="0.00001"/>
+      <mass value="0.000001"/>
       <inertia
-          ixx="0.000001" ixy="0.0" ixz="0.0"
-          iyy="0.000001" iyz="0.0"
-          izz="0.000002"/>
+          ixx="0.00000001" ixy="0.0" ixz="0.0"
+          iyy="0.00000001" iyz="0.0"
+          izz="0.00000002"/>
     </inertial>
   </link>
@@ -96,10 +96,10 @@
   <link name="main_body">
     <inertial>
-      <mass value = "0.832" />
+      <mass value = "0.0832" />
       <origin xyz="0.002 0 ${0.028 - 0.002}" rpy="0 0 0"/> <!-- TODO: true cog pos -->
       <inertia
-          ixx="0.0030" ixy="0" ixz="0"
-          iyy="0.0030" iyz="0"
-          izz="0.0045"/>
+          ixx="0.000030" ixy="0" ixz="0"
+          iyy="0.000030" iyz="0"
+          izz="0.000045"/>
     </inertial>
     <visual>
@@ -142,9 +142,9 @@
     <origin xyz="0.0 0 -0.035" rpy="${pi/2} 0 0"/>
     <inertial>
-      <mass value = "0.188" />
+      <mass value = "0.0188" />
       <origin xyz="0 0 0" rpy="0 0 0"/>
       <inertia
-          ixx="0.0002" ixy="0.0" ixz="0.0"
-          iyy="0.0002" iyz="0.0" izz="0.0002"/>
+          ixx="0.000002" ixy="0.0" ixz="0.0"
+          iyy="0.000002" iyz="0.0" izz="0.000002"/>
     </inertial>
   </xacro:extra_module>

Commit message: [mini_quadrotor] set half of small quadrotor in visualization and collision

File: robots/mini_quadrotor/urdf/robot.urdf.xacro (robot description, xacro)
@@ -58,5 +58,5 @@
         <origin rpy="0 0 0" xyz="0 0 0"/>
         <geometry>
-          <mesh filename="package://mini_quadrotor/urdf/mesh/prop_5inch.dae" />
+          <mesh filename="package://mini_quadrotor/urdf/mesh/prop_5inch.dae" scale="0.5 0.5 0.5"/>
         </geometry>
       </visual>
@@ -106,5 +106,5 @@
       <origin rpy="0 0 0" xyz="0 0 0"/>
       <geometry>
-        <mesh filename="package://mini_quadrotor/urdf/mesh/main_body_livox.dae" />
+        <mesh filename="package://mini_quadrotor/urdf/mesh/main_body_livox.dae" scale="0.5 0.5 0.5"/>
       </geometry>
     </visual>
@@ -112,5 +112,5 @@
       <origin rpy="0 0 0" xyz="0 0 0"/>
       <geometry>
-        <box size="0.28 0.28 0.072" />
+        <box size="0.14 0.14 0.072" />
       </geometry>
     </collision>
@@ -139,5 +139,5 @@
   </xacro:extra_module>
   <!-- battery -->
-  <xacro:extra_module name = "battery" parent = "main_body" visible = "1" model_url = "package://mini_quadrotor/urdf/mesh/turnigy_3S_2200mAh.dae" >
+  <xacro:extra_module name = "battery" parent = "main_body" visible = "1" model_url = "package://mini_quadrotor/urdf/mesh/turnigy_3S_2200mAh.dae" scale="0.5 0.5 0.5" >
     <origin xyz="0.0 0 -0.035" rpy="${pi/2} 0 0"/>
     <inertial>

Commit message: [mini_quadrotor] show black main quadrotor fig

File: robots/mini_quadrotor/urdf/robot.urdf.xacro (robot description, xacro)
@@ -106,5 +106,5 @@
       <origin rpy="0 0 0" xyz="0 0 0"/>
       <geometry>
-        <mesh filename="package://mini_quadrotor/urdf/mesh/main_body_livox.dae" scale="0.5 0.5 0.5"/>
+        <mesh filename="package://mini_quadrotor/urdf/mesh/main_body_livox_black.dae" scale="0.5 0.5 0.5"/>
       </geometry>
     </visual>

Commit message: [large_quadrotor] obstacle avoidance evaluation

File: robots/mini_quadrotor/urdf/robot.urdf.xacro (robot description, xacro)
@@ -6,7 +6,7 @@
   <thrust_link name="thrust" />
   <!-- kinematics [m] -->
-  <xacro:property name="rotor_x" value="0.035" />
-  <xacro:property name="rotor_y" value="0.035" />
-  <xacro:property name="rotor_z" value="0.010" />
+  <xacro:property name="rotor_x" value="0.1275" />
+  <xacro:property name="rotor_y" value="0.1275" />
+  <xacro:property name="rotor_z" value="0.039" />
   <!-- dynamics -->
   <m_f_rate value="-0.011" /> <!-- drag torque rate -->
@@ -49,14 +49,14 @@
       <inertial>
         <origin xyz="0 0 0" rpy="0 0 0"/>
-        <mass value="0.00091"/>
+        <mass value="0.03"/>
         <inertia
-            ixx="0.0000000807" ixy="0.0" ixz="0.0"
-            iyy="0.0000000807" iyz="0.0"
-            izz="0.0000001612"/>
+            ixx="0.0000607" ixy="0.0" ixz="0.0"
+            iyy="0.0000607" iyz="0.0"
+            izz="0.00012"/>
       </inertial>
       <visual>
         <origin rpy="0 0 0" xyz="0 0 0"/>
         <geometry>
-          <mesh filename="package://mini_quadrotor/urdf/mesh/prop_5inch.dae" scale="0.5 0.5 0.5"/>
+          <mesh filename="package://mini_quadrotor/urdf/mesh/prop_5inch.dae" scale="1.5 1.5 1.5"/>
         </geometry>
       </visual>
@@ -96,15 +96,15 @@
   <link name="main_body">
     <inertial>
-      <mass value = "0.0832" />
+      <mass value = "2.0" />
       <origin xyz="0.002 0 ${0.028 - 0.002}" rpy="0 0 0"/> <!-- TODO: true cog pos -->
       <inertia
-          ixx="0.000030" ixy="0" ixz="0"
-          iyy="0.000030" iyz="0"
-          izz="0.000045"/>
+          ixx="0.0220" ixy="0" ixz="0"
+          iyy="0.0220" iyz="0"
+          izz="0.0337"/>
     </inertial>
     <visual>
       <origin rpy="0 0 0" xyz="0 0 0"/>
       <geometry>
-        <mesh filename="package://mini_quadrotor/urdf/mesh/main_body_livox_black.dae" scale="0.5 0.5 0.5"/>
+        <mesh filename="package://mini_quadrotor/urdf/mesh/main_body_livox_black.dae" scale="1.5 1.5 1.5"/>
       </geometry>
     </visual>
@@ -112,5 +112,5 @@
       <origin rpy="0 0 0" xyz="0 0 0"/>
       <geometry>
-        <box size="0.14 0.14 0.072" />
+        <box size="0.42 0.42 0.072" />
       </geometry>
     </collision>
@@ -139,12 +139,12 @@
   </xacro:extra_module>
   <!-- battery -->
-  <xacro:extra_module name = "battery" parent = "main_body" visible = "1" model_url = "package://mini_quadrotor/urdf/mesh/turnigy_3S_2200mAh.dae" scale="0.5 0.5 0.5" >
+  <xacro:extra_module name = "battery" parent = "main_body" visible = "1" model_url = "package://mini_quadrotor/urdf/mesh/turnigy_3S_2200mAh.dae" scale="1.5 1.5 1.5" >
     <origin xyz="0.0 0 -0.035" rpy="${pi/2} 0 0"/>
     <inertial>
-      <mass value = "0.0188" />
+      <mass value = "0.282" />
       <origin xyz="0 0 0" rpy="0 0 0"/>
       <inertia
-          ixx="0.000002" ixy="0.0" ixz="0.0"
-          iyy="0.000002" iyz="0.0" izz="0.000002"/>
+          ixx="0.0003" ixy="0.0" ixz="0.0"
+          iyy="0.0003" iyz="0.0" izz="0.0003"/>
     </inertial>
   </xacro:extra_module>
