Commit message: [agile_multirotor] shift CoG position

File: robots/agile_multirotor/urdf/quadrotor.urdf.xacro (robot description, xacro)
@@ -193,5 +193,22 @@
   <xacro:include filename="$(find hector_sensors_description)/urdf/hokuyo_utm30lx.urdf.xacro" />
   <xacro:hokuyo_utm30lx_model name="laser" parent="main_body">
-    <origin xyz="0.0 0.0 0.076" rpy="0 0 0"/>
+    <origin xyz="0.20 0.0 0.076" rpy="0 0 0"/>
   </xacro:hokuyo_utm30lx_model>
+  <joint name="dummy_joint" type="fixed">
+    <parent link="main_body"/>
+    <child link="dummy_body"/>
+    <origin rpy="0 0 0" xyz="0.1 0 0"/>
+    <axis xyz="0 0 1"/>
+  </joint>
+  <!-- dummy_body -->
+  <link name="dummy_body">
+    <inertial>
+      <mass value = "0.3" />
+      <origin xyz="0.0 0.0 0.0" rpy="0 0 0"/>
+      <inertia
+          ixx="0.00001" ixy="0.0000" ixz="0.0000"
+          iyy="0.00001" iyz="0.00000"
+          izz="0.00001"/>
+    </inertial>
+  </link>
 </robot>
